File: src/devices/Seatalk1/schematics/SeaTalk1/SeaTalk1.kicad_pcb (KiCad board)
At the start: 2 copper layers, 0 parts

Commit message: Minor cleanup, create empty PCB
Parts:
- added C1: 150u, Capacitor_THT:CP_Radial_D12.5mm_P7.50mm, F.Cu at (83.9, 91.4)
- added D1: LED, LED_THT:LED_D3.0mm_Horizontal_O3.81mm_Z6.0mm, F.Cu at (85.7, 48.7)
- added J1: Raspberry_Pi_2_3, Connector_PinSocket_2.54mm:PinSocket_2x20_P2.54mm_Vertical, F.Cu at (132.1, 48.3)
- added J3: Conn_01x03_Pin, Connector_PinHeader_2.54mm:PinHeader_1x03_P2.54mm_Vertical, F.Cu at (40.6, 86.4)
- added Q1: BC557, Package_TO_SOT_THT:TO-92_Inline, F.Cu at (79.4, 50.2)
- added Q2: BC547, Package_TO_SOT_THT:TO-92_Inline, F.Cu at (79.4, 56.0)
- added Q3: BC547, Package_TO_SOT_THT:TO-92_Inline, F.Cu at (79.4, 61.8)
- added Q4: BC547, Package_TO_SOT_THT:TO-92_Inline, F.Cu at (79.4, 67.5)
- added Q5: BC547, Package_TO_SOT_THT:TO-92_Inline, F.Cu at (79.4, 73.3)
- added Q6: BC547, Package_TO_SOT_THT:TO-92_Inline, F.Cu at (79.4, 79.1)
- added R1: 22k, Resistor_THT:R_Axial_DIN0309_L9.0mm_D3.2mm_P15.24mm_Horizontal, F.Cu at (53.4, 49.3)
- added R10: 1.5k, Resistor_THT:R_Axial_DIN0309_L9.0mm_D3.2mm_P15.24mm_Horizontal, F.Cu at (53.4, 92.0)
- added R13: 10k, Resistor_THT:R_Axial_DIN0309_L9.0mm_D3.2mm_P15.24mm_Horizontal, F.Cu at (53.4, 96.8)
- added R14: 2.2k, Resistor_THT:R_Axial_DIN0309_L9.0mm_D3.2mm_P15.24mm_Horizontal, F.Cu at (53.4, 101.5)
- added R15: 10k, Resistor_THT:R_Axial_DIN0309_L9.0mm_D3.2mm_P15.24mm_Horizontal, F.Cu at (53.4, 106.3)
- added R2: 2.2k, Resistor_THT:R_Axial_DIN0309_L9.0mm_D3.2mm_P15.24mm_Horizontal, F.Cu at (53.4, 54.0)
- added R3: 2.2k, Resistor_THT:R_Axial_DIN0309_L9.0mm_D3.2mm_P15.24mm_Horizontal, F.Cu at (53.4, 58.8)
- added R4: 4.7k, Resistor_THT:R_Axial_DIN0309_L9.0mm_D3.2mm_P15.24mm_Horizontal, F.Cu at (53.4, 63.5)
- added R5: 4.7k, Resistor_THT:R_Axial_DIN0309_L9.0mm_D3.2mm_P15.24mm_Horizontal, F.Cu at (53.4, 68.3)
- added R6: 4.7k, Resistor_THT:R_Axial_DIN0309_L9.0mm_D3.2mm_P15.24mm_Horizontal, F.Cu at (53.4, 73.0)
- added R7: 22k, Resistor_THT:R_Axial_DIN0309_L9.0mm_D3.2mm_P15.24mm_Horizontal, F.Cu at (53.4, 77.8)
- added R8: 2.2k, Resistor_THT:R_Axial_DIN0309_L9.0mm_D3.2mm_P15.24mm_Horizontal, F.Cu at (53.4, 82.5)
- added R9: 100, Resistor_THT:R_Axial_DIN0309_L9.0mm_D3.2mm_P15.24mm_Horizontal, F.Cu at (53.4, 87.3)

Commit message: Schema updated, PCB drawn (unverified!)
Parts:
- added R12: 10k, Resistor_THT:R_Axial_DIN0207_L6.3mm_D2.5mm_P10.16mm_Horizontal, F.Cu at (99.0, 96.0)
- D1: value LED -> blue
- J1: moved to B.Cu
- R1, R10, R13, R14, R15, R2, R3, R4, R5, R6, R7, R8, R9: footprint Resistor_THT:R_Axial_DIN0309_L9.0mm_D3.2mm_P15.24mm_Horizontal -> Resistor_THT:R_Axial_DIN0207_L6.3mm_D2.5mm_P10.16mm_Horizontal
- moved R1 66.0 mm to (114.5, 74.2), turned to 90 degrees
- moved R14 60.7 mm to (107.0, 73.0), turned to -90 degrees
- moved R3 60.2 mm to (113.1, 51.0), turned to 180 degrees
- moved R7 57.8 mm to (111.0, 72.9), turned to -90 degrees
- moved D1 54.3 mm to (115.8, 93.9)
- moved R8 51.0 mm to (104.0, 76.0), turned to 180 degrees
- moved R9 50.9 mm to (102.9, 99.0)
- moved R13 50.6 mm to (104.0, 95.0), turned to 90 degrees
- moved Q3 47.3 mm to (117.7, 89.4)
- moved R5 46.6 mm to (98.1, 55.0), turned to 180 degrees
- moved R2 44.7 mm to (98.0, 51.0), turned to 180 degrees
- moved J3 43.6 mm to (84.0, 90.5)
- moved R10 41.4 mm to (93.4, 81.5)
- moved Q4 40.7 mm to (117.7, 81.0)
- moved Q6 40.1 mm to (118.0, 68.4)
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Routing:
- net VCC_3.3: track 0.00 -> 101.2 mm
- net GND: track 0.00 -> 95.3 mm
- net SEATALK: track 0.00 -> 87.2 mm
- net TXD: track 0.00 -> 69.1 mm
- net Net-(Q4-B): track 0.00 -> 51.4 mm
- net Net-(J1-GPIO15/RXD): track 0.00 -> 47.7 mm
- net Net-(Q5-C): track 0.00 -> 46.5 mm
- net Net-(Q2-B): track 0.00 -> 45.3 mm
- net VCC_5.0: track 0.00 -> 39.7 mm
- net Net-(Q1-B): track 0.00 -> 37.0 mm
- net Net-(C1-Pad1): track 0.00 -> 31.6 mm
- net Net-(Q5-B): track 0.00 -> 10.4 mm
- net Net-(D1-A): track 0.00 -> 7.92 mm
- net Net-(D1-K): track 0.00 -> 5.86 mm
- net Net-(J3-Pin_3): track 0.00 -> 5.03 mm
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- added copper zone on B.Cu, net GND
Other:
- board outline added: 56 x 65 mm

Commit message: Documentation started
Connections:
- J1 pad 10: Net-(J1-GPIO15/RXD) -> unconnected-(J1-GPIO15/RXD-Pad10)
- J1 pad 27: unconnected-(J1-ID_SD/GPIO0-Pad27) -> TXD
- J1 pad 28: unconnected-(J1-ID_SC/GPIO1-Pad28) -> Net-(J1-ID_SC/GPIO1)
- J1 pad 8: TXD -> unconnected-(J1-GPIO14/TXD-Pad8)
- Q2 pad 1: Net-(J1-GPIO15/RXD) -> Net-(J1-ID_SC/GPIO1)
- R8 pad 2: Net-(J1-GPIO15/RXD) -> Net-(J1-ID_SC/GPIO1)
Routing:
- net Net-(J1-ID_SC/GPIO1): track 0.00 -> 66.0 mm
- net Net-(J1-GPIO15/RXD): track 47.7 -> 0.00 mm
- net GND: track 95.3 -> 60.3 mm
- net TXD: track 69.1 -> 57.6 mm
- net Net-(Q5-B): track 10.4 -> 11.7 mm
